File: PCB/FT817_buddy_v4/FT817_buddy_v4.kicad_sch (KiCad schematic)
At the start: 65 parts, among them J1 FT817_ACC, J2 KEY_OUT, J3 KEY_IN, J4 K16 CW processor, J5 GND, J6 EXP PWR SELECT, J7 , J8 , J9 EXPANSION HEADER, SW1 SW_Push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

Commit message: updaten schematic and pcb
Parts:
- J7, J8: value (none) -> (none)
Other:
- note added: "Display"
